File: hardware/ext-board/ext-board.kicad_pcb (KiCad board)
At the start: 2 copper layers, 38.5 x 85 mm, 24 parts, among them J1 GH BM07B link to INT, J2 VCC DATA GND, J3 PTSM 0,5/2-HH-2,5-THR 24 VAC, J4 5V OUT to Pi USB-C, U1 DS2482-100, U2 DS2482-100 (0x19), U3 TMR 12-4811WI

Commit message: INT: J6's pin legend on the front silkscreen beside the pads; the back-side legend served a through-hole header
Co-Authored-By: Claude Fable 5.1 <noreply@anthropic.com>
Routing:
- net VCC: track 162.3 -> 190.9 mm, vias 2 -> 1
- net GND: track 203.5 -> 175.8 mm, vias 2 -> 1
- net DATA: track 115.2 -> 137.3 mm, vias 0 -> 1
- net H3_DATA: track 22.2 -> 15.6 mm
- net SDA: track 74.9 -> 80.6 mm
- net COM: track 47.0 -> 52.0 mm
- net ACF: track 34.0 -> 29.1 mm
- net ACR: track 43.3 -> 39.7 mm
- net SCL: track 74.4 -> 76.8 mm, vias 2 -> 0
- net VS: track 82.8 -> 84.9 mm

Commit message: Silkscreen: INT header pin numbers on their pins, J9 above its column, J5's back reference hidden; EXT probe-end labels aligned
Co-Authored-By: Claude Fable 5.1 <noreply@anthropic.com>
Routing:
- net VCC: track 190.9 -> 150.0 mm, vias 1 -> 3
- net ACR: track 39.7 -> 54.0 mm
- net VS: track 84.9 -> 72.6 mm, vias 0 -> 1
- net DATA: track 137.3 -> 146.1 mm, vias 1 -> 0
- net GND: track 175.8 -> 167.1 mm
- net SDA: track 80.6 -> 75.1 mm
- net ACF: track 29.1 -> 34.0 mm
- net COM: track 52.0 -> 48.7 mm, vias 1 -> 0
- net SCL: track 76.8 -> 74.4 mm, vias 0 -> 2
- net ACC: track 60.7 -> 60.6 mm, vias 0 -> 1
Other:
- board text added: "D"
- board text added: "G"
- board text added: "V"
- board text removed: "V D G"
