File: hardware/ext-board/ext-board.kicad_sch (KiCad schematic)
At the start: 12 parts, among them J1 LINK to INT, J2 bus pads, U1 DS2482-100 (0x18), U2 DS2482-100 (0x19, not fitted)

Commit message: Rev B boards generated: KiCad, schematics, BOMs and OSH Park gerbers for INT and EXT
gen-boards.py now builds rev B. INT loses the bridge, F1, C1, J7 and J8,
J4 carries HPCOOL, DHWX and SP-E, the sockets sit at x 13 with the resistor
columns on 4.0 mm (the most the housing bulges' rule areas allow), J6 is the
JST GH side-entry header at the slot with VS and COM on pins 6 and 7, and the
DL title block is centred in the bottom field. EXT keeps the probe sockets,
puts the I2C parts in one row under them, and carries the power section:
J3 24 VAC entry at the bottom edge with the sockets' 1.7 mm overhang, F1
standing, D1-D4 at 3.5 mm rows, C3 standing, U3 on a new SIP-8 footprint,
C4, J4 (XH) for the USB-C pigtail, a tie-slot pair, a 6 x 4 proto field and
the GH top-entry link header low at the opening, pin 1 at the bottom on both
boards. Freerouting is not deterministic, so build.sh regenerates and reroutes
each board until DRC is clean and everything is connected; five connections
it kept leaving open are laid as fixed tracks. Both boards are DRC-clean with
nothing unconnected; build.sh now also exports the gerbers and drill files
and zips them.

The plan carries the generated numbers and the state of the build; the layout
SVG matches it.

Co-Authored-By: Claude Fable 5.1 <noreply@anthropic.com>
Parts:
- removed J1: LINK to INT, pivac:PTSM_0.5_5-HH-2.5-THR, symbol Connector_Generic:Conn_01x05
- added C3: 470u 63V, Capacitor_THT:CP_Radial_D12.5mm_P5.00mm, symbol Device:C_Polarized
- added C4: 1u, Capacitor_THT:C_Rect_L7.0mm_W2.5mm_P5.00mm, symbol Device:C
- added D1, D2, D3, D4: 1N4007, Diode_THT:D_DO-41_SOD81_P10.16mm_Horizontal, symbol Device:D
- added F1: PTC 1.1A 60V, pivac:PTC_Radial_P5.08_Standing, symbol Device:Fuse
- added J1: GH link to INT, Connector_JST:JST_GH_BM07B-GHS-TBT_1x07-1MP_P1.25mm_Vertical, symbol Connector_Generic:Conn_01x07
- added J3: PTSM 0,5/2-HH 24 VAC, pivac:PTSM_0.5_2-HH-2.5-THR, symbol Connector_Generic:Conn_01x02
- added J4: XH 5V OUT to Pi USB-C, Connector_JST:JST_XH_B2B-XH-A_1x02_P2.50mm_Vertical, symbol Connector_Generic:Conn_01x02
- added U3: TMR 12-4811WI, pivac:TMR12WI_SIP-8, symbol pivac:TMR12WI
Connections:
- net GND: now also C4.2, J1.5 (Pin_5), J4.2 (Pin_2), U3.7 (-Vout)
- net GPIO4: now also J1.4 (Pin_4)
- net SCL: now also J1.3 (Pin_3)
- net SDA: now also J1.2 (Pin_2)
- net VCC: now also J1.1 (Pin_1)
- new net +5V: C4.1, J4.1 (Pin_1), U3.6 (+Vout)
- new net ACC: D2.2 (A), D4.1 (K), J3.2 (Pin_2)
- new net ACF: D1.2 (A), D3.1 (K), F1.2
- new net ACR: F1.1, J3.1 (Pin_1)
- new net COM: C3.2, D3.2 (A), D4.2 (A), J1.7 (Pin_7), U3.1 (-Vin)
- new net VS: C3.1, D1.1 (K), D2.1 (K), J1.6 (Pin_6), U3.2 (+Vin)
- no-connect marks 2 -> 4
Other:
- note added: "24 VAC in on J3, PTC F1, bridge D1-D4, C3 470 uF: VS about 35 V DC against COM, out to INT on J1.6/J1.7 and into U3."
- note added: "U3 makes 5.1 V isolated for the Pi: C4 at its output, J4 to a USB-C pigtail. Remote (pin 3) open = on. COM never meets GND."
- note added: "pivac EXT board rev B: DS2482-100 1-wire master, three probe sockets, 24 VAC sense supply and the Pi's 5.1 V supply, link to the INT board"
- note removed: "pivac EXT board rev A: DS2482-100 1-wire master, three probe sockets, link to the INT board"
