File: hardware/ext-board/ext-board.kicad_sch (KiCad schematic)
At the start: 12 parts, among them J1 LINK to INT, J2 bus pads, U1 DS2482-100 (0x18), U2 DS2482-100 (0x19, not fitted)

Commit message: Rev B plan: Pi supply on EXT, GH link, every channel on a plug (#214)
* Rev B plan: the Pi's supply moves to the EXT board, GH link, every channel on a plug

Rev A left the Pi on a wall adapter and put the 24 VAC entry on INT, which cost
two plug positions and forced HPCOOL onto the J8 pigtail whose loose connector
was the one fault at the 2026-09-26 cutover. Rev B moves the entry, the PTC, the
bridge and the reservoir to EXT's mid field, adds an isolated Traco TMR 12-4811WI
there, and feeds the Pi's own USB-C by a pigtail from a 2-pin XH header, so the
Pi's input protection stays in circuit and header pins 2 and 4 carry nothing.
VS and COM come back to INT over a 7-way JST GH link that replaces the PTSM
J6/J7 pair and latches after the boards are seated. J4 then takes HPCOOL, DHWX
and SP-E, J8 goes away, the optocoupler sockets shift right to clear the J9
breakout, and both boards get a DL title block.

The plan doc carries the circuit, the link pin map, the plug map, the EXT
positions, the parts list with distributor links and the path to the OSH Park
order. The SVG is the layout for review at 8 px per mm; hardware/dl-monogram.svg
is the mark's source for the KiCad footprint. The PCB plan's power section and
open items now state the rev B position.

Co-Authored-By: Claude Fable 5.1 <noreply@anthropic.com>

* Rev B plan: component index for both boards, PTSM edge offsets, link header at the rib

The plan now names every reference designator on both boards with its part,
body size, position and purpose, states how each PTSM header meets its board
edge (pin row 5.4 mm behind the entry face, from the Phoenix drawing the
footprint is built from: INT plugs 1.55 mm inside, EXT sockets and J3 1.7 mm
outside), and carries the carried-over parts alongside the new ones. EXT's J1
moves down to y 46.5-58.5 so it does not sit opposite INT's J6 in the opening.
The layout SVG draws the PTSM bodies at those offsets and J1 at its new place.

Co-Authored-By: Claude Fable 5.1 <norepl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
Parts:
- removed J1: LINK to INT, pivac:PTSM_0.5_5-HH-2.5-THR, symbol Connector_Generic:Conn_01x05
- added C3: 470u 63V, Capacitor_THT:CP_Radial_D12.5mm_P5.00mm, symbol Device:C_Polarized
- added C4: 1u, Capacitor_THT:C_Rect_L7.0mm_W2.5mm_P5.00mm, symbol Device:C
- added D1, D2, D3, D4: 1N4007, Diode_THT:D_DO-41_SOD81_P10.16mm_Horizontal, symbol Device:D
- added F1: PTC 1.1A 60V, pivac:PTC_Radial_P5.08_Standing, symbol Device:Fuse
- added J1: GH link to INT, Connector_JST:JST_GH_BM07B-GHS-TBT_1x07-1MP_P1.25mm_Vertical, symbol Connector_Generic:Conn_01x07
- added J3: PTSM 0,5/2-HH 24 VAC, pivac:PTSM_0.5_2-HH-2.5-THR, symbol Connector_Generic:Conn_01x02
- added J4: XH 5V OUT to Pi USB-C, Connector_JST:JST_XH_B2B-XH-A_1x02_P2.50mm_Vertical, symbol Connector_Generic:Conn_01x02
- added U3: TMR 12-4811WI, pivac:TMR12WI_SIP-8, symbol pivac:TMR12WI
Connections:
- net GND: now also C4.2, J1.5 (Pin_5), J4.2 (Pin_2), U3.7 (-Vout)
- net GPIO4: now also J1.4 (Pin_4)
- net SCL: now also J1.3 (Pin_3)
- net SDA: now also J1.2 (Pin_2)
- net VCC: now also J1.1 (Pin_1)
- new net +5V: C4.1, J4.1 (Pin_1), U3.6 (+Vout)
- new net ACC: D2.2 (A), D4.1 (K), J3.2 (Pin_2)
- new net ACF: D1.2 (A), D3.1 (K), F1.2
- new net ACR: F1.1, J3.1 (Pin_1)
- new net COM: C3.2, D3.2 (A), D4.2 (A), J1.7 (Pin_7), U3.1 (-Vin)
- new net VS: C3.1, D1.1 (K), D2.1 (K), J1.6 (Pin_6), U3.2 (+Vin)
- no-connect marks 2 -> 4
Other:
- note added: "24 VAC in on J3, PTC F1, bridge D1-D4, C3 470 uF: VS about 35 V DC against COM, out to INT on J1.6/J1.7 and into U3."
- note added: "U3 makes 5.1 V isolated for the Pi: C4 at its output, J4 to a USB-C pigtail. Remote (pin 3) open = on. COM never meets GND."
- note added: "pivac EXT board rev B: DS2482-100 1-wire master, three probe sockets, 24 VAC sense supply and the Pi's 5.1 V supply, link to the INT board"
- note removed: "pivac EXT board rev A: DS2482-100 1-wire master, three probe sockets, link to the INT board"
