File: hardware/int-board/int-board.kicad_sch (KiCad schematic)
At the start: 33 parts, among them J1 PTSM 0,5/4-HH, J2 PTSM 0,5/4-HH, J3 PTSM 0,5/4-HH, J4 PTSM 0,5/4-HH, J5 Pi 40-pin socket, J6 LINK to EXT, J7 PWR link (not fitted), J8 spare ch pads, J9 breakout, U1 LTV-847, U2 LTV-847, U3 LTV-847

Commit message: Rev B plan: Pi supply on EXT, GH link, every channel on a plug (#214)
* Rev B plan: the Pi's supply moves to the EXT board, GH link, every channel on a plug

Rev A left the Pi on a wall adapter and put the 24 VAC entry on INT, which cost
two plug positions and forced HPCOOL onto the J8 pigtail whose loose connector
was the one fault at the 2026-09-26 cutover. Rev B moves the entry, the PTC, the
bridge and the reservoir to EXT's mid field, adds an isolated Traco TMR 12-4811WI
there, and feeds the Pi's own USB-C by a pigtail from a 2-pin XH header, so the
Pi's input protection stays in circuit and header pins 2 and 4 carry nothing.
VS and COM come back to INT over a 7-way JST GH link that replaces the PTSM
J6/J7 pair and latches after the boards are seated. J4 then takes HPCOOL, DHWX
and SP-E, J8 goes away, the optocoupler sockets shift right to clear the J9
breakout, and both boards get a DL title block.

The plan doc carries the circuit, the link pin map, the plug map, the EXT
positions, the parts list with distributor links and the path to the OSH Park
order. The SVG is the layout for review at 8 px per mm; hardware/dl-monogram.svg
is the mark's source for the KiCad footprint. The PCB plan's power section and
open items now state the rev B position.

Co-Authored-By: Claude Fable 5.1 <noreply@anthropic.com>

* Rev B plan: component index for both boards, PTSM edge offsets, link header at the rib

The plan now names every reference designator on both boards with its part,
body size, position and purpose, states how each PTSM header meets its board
edge (pin row 5.4 mm behind the entry face, from the Phoenix drawing the
footprint is built from: INT plugs 1.55 mm inside, EXT sockets and J3 1.7 mm
outside), and carries the carried-over parts alongside the new ones. EXT's J1
moves down to y 46.5-58.5 so it does not sit opposite INT's J6 in the opening.
The layout SVG draws the PTSM bodies at those offsets and J1 at its new place.

Co-Authored-By: Claude Fable 5.1 <norepl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
Parts:
- removed C1: 100u 63V axial, Capacitor_THT:CP_Axial_L18.0mm_D6.5mm_P25.00mm_Horizontal, symbol Device:C_Polarized
- removed D1, D2, D3, D4: 1N4007, Diode_THT:D_DO-41_SOD81_P10.16mm_Horizontal, symbol Device:D
- removed F1: PTC 0.1A 60V, pivac:PTC_Radial_P5.08_Flat, symbol Device:Fuse
- removed J6: LINK to EXT, pivac:PTSM_0.5_5-HH-2.5-THR, symbol Connector_Generic:Conn_01x05
- removed J7: PWR link (not fitted), pivac:PTSM_0.5_4-HH-2.5-THR, symbol Connector_Generic:Conn_01x04
- removed J8: spare ch pads, pivac:Pads_3x1, symbol Connector_Generic:Conn_01x03
- added J6: GH link to EXT, Connector_JST:JST_GH_SM07B-GHS-TB_1x07-1MP_P1.25mm_Horizontal, symbol Connector_Generic:Conn_01x07
Connections:
- net S_SP-C is gone; now on net S_DHWX: R11.2
- net 3V3: now also J6.1 (Pin_1)
- net COM: now also J6.7 (Pin_7)
- net GND: now also J6.5 (Pin_5)
- net GPIO13: now also U3.14 (C2); no longer U3.12 (C3)
- net GPIO19: now also U3.12 (C3); no longer U3.14 (C2)
- net GPIO4: now also J6.4 (Pin_4)
- net SCL: now also J6.3 (Pin_3)
- net SDA: now also J6.2 (Pin_2)
- net S_SP-E: now also J4.3 (Pin_3)
- net VS: now also J6.6 (Pin_6)
- net ACC renamed S_DHWX
- net ACR renamed S_HPCOOL
- net S_HPCOOL: now also R10.2
- removed net S_SP-D: J4.3 (Pin_3), R10.2
Other:
- note added: "Field plugs, PTSM 0,5/4-HH-2,5-THR; position 4 is COM on every plug; twelve channels on twelve positions"
- note added: "J4.1 > G13 (p33)"
- note added: "J4.2 > G19 (p35)"
- note added: "J4.3 > G16 (p36)"
- note added: "Shadow column J9: one pad per header row (rows 1, 2, 16, 18 empty); pins 2 and 4 (5 V) carry nothing, the Pi is fed by USB-C"
- note added: "The sense supply (VS about 35 V DC, COM its return) is made on the EXT board and arrives on J6.6/J6.7."
- note added: "ch10 HPCOOL"
- note added: "ch11 DHWX"
- note added: "pivac INT board rev B: relay-sense inputs on LTV-847 optocouplers; VS/COM arrive from the EXT board"
- note removed: "24 VAC sense supply: PTC, full-wave bridge, 100 uF; VS is about 35 V DC, COM its return; C1 and F1 lie flat, nothing on the component side stands over 8 mm"
- note removed: "Field plugs, PTSM 0,5/4-HH-2,5-THR; position 4 is COM on every plug; J4.1/J4.2 take the 24 VAC"
- note removed: "J4.3 > G19 (p35)"
- note removed: "J8 > G13 (p33)"
- note removed: "J8 > G16 (p36)"
- note removed: "Shadow column J9: one pad per header row (rows 1, 2, 16, 18 empty)"
- note removed: "ch10 SP-D"
- note removed: "ch11 SP-C"
- note removed: "pivac INT board rev A: relay-sense inputs on LTV-847 optocouplers, 24 VAC sense supply"
