File: hardware/int-board/int-board.kicad_sch (KiCad schematic)
At the start: 25 parts, among them J1 PTSM 0,5/4-HH, J2 PTSM 0,5/4-HH, J3 PTSM 0,5/4-HH, J4 PTSM 0,5/4-HH, J5 Pi 40-pin socket, J6 GH link to EXT, J9 breakout, U1 LTV-847, U2 LTV-847, U3 LTV-847

Commit message: Rev B INT: 10 kΩ LED resistors in place of 12 kΩ
The resistor assortment on hand has 10 kΩ and 22 kΩ but no 12 kΩ. 10 kΩ
sets 3.4 mA per channel from the 35 V sense rail (0.11 W, under half the
1/4 W rating, far under the LTV-847's 50 mA), adds 7 mA to the bridge with
all twelve channels on, and keeps the relay contacts at a higher wetting
current. 22 kΩ would drop to about 1 mA at 21.6 VAC under the Pi's load,
half the current any build has proven.

The value appears in no gerber layer, so the ordered boards are unchanged;
the generated BOM, schematic and KiCad files are edited in place rather
than rebuilt, which would reroute the board. Rev A keeps its 12 kΩ.

Co-Authored-By: Claude Opus 5.5 <noreply@anthropic.com>
Parts:
- R1, R10, R11, R12, R2, R3, R4, R5, R6, R7, R8, R9: value 12k 1/4W -> 10k 1/4W
