File: hardware/ah-board/ah-board.kicad_pcb (KiCad board)
At the start: 2 copper layers, 86.4 x 53.3 mm, 54 parts, among them J1 test row, J10 Arduino header, J11 Arduino header, J12 Arduino header, J13 Arduino header, U1 TMR 3-4811WI, U2 DS2482S-100+, U3 LTV-814S, U4 LTV-814S

Commit message: Air-handler shield: no ICSP holes
On the proto shield the R4's barrel jack (11 mm, plastic) holds the shield
above the ICSP pins (8.5 mm), so the six clearance holes and their keep-out
do nothing. They are removed, which also drops the ICSP position from the
checks before ordering. No insulation is needed over the jack's plastic
shell.

Co-Authored-By: Claude Opus 5.5 <noreply@anthropic.com>
Parts:
- removed H1: ICSP clearance, pivac:ICSP_Clearance_2x3
Routing:
- net OWD: track 121.9 -> 60.2 mm, vias 1 -> 2
- net OWV: track 97.9 -> 52.9 mm, vias 1 -> 2
- net GND: track 318.1 -> 275.2 mm
- net COM: track 82.2 -> 119.7 mm, vias 1 -> 3
- net ACF: track 40.1 -> 52.3 mm
- net SDA: track 98.5 -> 86.4 mm
- net SCL: track 99.3 -> 110.2 mm, vias 2 -> 1
- net +5V: track 213.7 -> 207.3 mm
- net Y2A: track 4.58 -> 9.29 mm
- net A0: track 74.2 -> 78.7 mm
- net D2: track 44.0 -> 39.9 mm
- net Y2C: track 25.6 -> 29.2 mm
- net D8: track 69.6 -> 66.2 mm
- net W2C: track 24.0 -> 27.4 mm
- net VS: track 24.7 -> 27.6 mm
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